Commit message: 一通り動くように。

File: my_robo_description/urdf/camera/d435.gazebo.xacro (robot description, xacro)
@@ -22,10 +22,10 @@
           <alwaysOn>true</alwaysOn>
           <updateRate>0.0</updateRate>
-          <imageTopicName>d435/image_raw</imageTopicName>
-          <cameraInfoTopicName>d435/camera_info</cameraInfoTopicName>
-          <depthImageTopicName>d435/depth/image_raw</depthImageTopicName>
+          <imageTopicName>d435/color/image_raw</imageTopicName>
+          <cameraInfoTopicName>d435/color/camera_info</cameraInfoTopicName>
+          <depthImageTopicName>d435/aligned_depth_to_color/image_raw</depthImageTopicName>
           <depthImageCameraInfoTopicName>d435/depth/camera_info</depthImageCameraInfoTopicName>
-          <pointCloudTopicName>d435/depth/points</pointCloudTopicName>
-          <frameName>d435_link_optical</frameName>
+          <pointCloudTopicName>d435/depth/color/points</pointCloudTopicName>
+          <frameName>d435_color_optical_frame</frameName>
           <pointCloudCutoff>0.01</pointCloudCutoff>
           <pointCloudCutoffMax>15.0</pointCloudCutoffMax>

File: my_robo_description/urdf/camera/d435.urdf.xacro (robot description, xacro)
@@ -1,5 +1,5 @@
 <robot
   xmlns:xacro="http://ros.org/wiki/xacro">
-  <xacro:macro name="d435" params="parent xyz">
+  <xacro:macro name="d435" params="parent xyz isSimulator">
     <xacro:include filename="$(find my_robo_description)/urdf/camera/d435.gazebo.xacro"/>
     <link name="d435_link">
@@ -26,14 +26,16 @@
       <child link="d435_link" />
     </joint>
-    <link name="d435_link_optical"/>
-    <joint name="d435_link_to_d435_link_optical_joint" type="fixed">
-      <!-- these values have to be these values otherwise the gazebo camera
+    <xacro:if value="${isSimulator}">
+      <link name="d435_color_optical_frame"/>
+      <joint name="d435_link_to_d435_color_optical_frame_joint" type="fixed">
+        <!-- these values have to be these values otherwise the gazebo camera
         image won't be aligned properly with the frame it is supposedly
         originating from -->
-      <!--https://answers.ros.org/question/232534/gazebo-camera-frame-is-inconsistent-with-rviz-opencv-convention/?answer=232562#post-id-232562-->
-      <origin xyz="0 0 0" rpy="${-pi/2} 0 ${-pi/2}"/>
-      <parent link="d435_link"/>
-      <child link="d435_link_optical"/>
-    </joint>
+        <!--https://answers.ros.org/question/232534/gazebo-camera-frame-is-inconsistent-with-rviz-opencv-convention/?answer=232562#post-id-232562-->
+        <origin xyz="0 0 0" rpy="${-pi/2} 0 ${-pi/2}"/>
+        <parent link="d435_link"/>
+        <child link="d435_color_optical_frame"/>
+      </joint>
+    </xacro:if>
   </xacro:macro>
 </robot>

File: my_robo_description/urdf/my_robo.urdf.xacro (robot description, xacro)
@@ -78,5 +78,5 @@
     <child link="body_link" />
   </joint>
-  <xacro:d435 parent="body_link" xyz="0.51 0 0.5"/>
+  <xacro:d435 parent="body_link" xyz="0.51 0 0.5" isSimulator="$(arg isSimulator)"/>
   <crane_plus parent="body_link"
               servo_color="black" bracket_color="grey" gripper_color="black"
@@ -90,4 +90,6 @@
     <plugin name="gazebo_ros_control" filename="libgazebo_ros_control.so"></plugin>
   </gazebo>
-  <xacro:d435_gazebo/>
+  <xacro:if value="$(arg isSimulator)">
+    <xacro:d435_gazebo/>
+  </xacro:if>
 </robot>
